File: hardware/ESR Meter v6.brd (EAGLE design)
At the start: 80 x 36 mm, 34 parts, among them Q1 MOSFET-NCHANNELFQP30N06L, U1 ATMEGA328P, U2 3V3, U3 LM317, Y1 8M

Commit message: Update library used for L4931
Parts:
- U2: device RBBB:L4931 -> l4931:L4931
Changed lines of the file:
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@@
 <attribute name="NAME" x="43.561" y="25.654" size="1.27" layer="25" font="vector" ratio="10"/>
 </element>
-<element name="U2" library="RBBB" package="L4931" value="3V3" x="49.53" y="26.67" smashed="yes" rot="R90">
+<element name="U2" library="l4931" package="L4931" value="3V3" x="49.53" y="26.67" smashed="yes" rot="R90">
 <attribute name="NAME" x="50.8" y="31.4452" size="1.27" layer="25" font="vector" ratio="10" rot="R180"/>
 </element>

Commit message: Rewrote README.md
Parts:
- R8: value 1 -> 1 1%
Changed lines of the file:
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@@
 <attribute name="NAME" x="74.041" y="27.559" size="1.27" layer="25" font="vector" ratio="10"/>
 </element>
-<element name="R8" library="resistor" package="0617V" value="1" x="76.835" y="21.59" smashed="yes" rot="R270">
+<element name="R8" library="resistor" package="0617V" value="1 1%" x="76.835" y="21.59" smashed="yes" rot="R270">
 <attribute name="NAME" x="73.66" y="23.6474" size="1.27" layer="25" font="vector" ratio="10"/>
 <attribute name="VALUE" x="74.2188" y="20.955" size="1.27" layer="27" font="vector" ratio="10" rot="R270"/>

Commit message: Edited README
Parts:
- Q1: value MOSFET-NCHANNELFQP30N06L -> FQP30N06L
Changed lines of the file:
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@@
 </element>
 <element name="LOGO1" library="SparkFun-Aesthetics" package="OSHW-LOGO-M" value="OSHW-LOGOM" x="73.66" y="7.62" smashed="yes"/>
-<element name="Q1" library="SparkFun-DiscreteSemi" package="TO220V" value="MOSFET-NCHANNELFQP30N06L" x="69.85" y="26.67" smashed="yes" rot="R270">
+<element name="Q1" library="SparkFun-DiscreteSemi" package="TO220V" value="FQP30N06L" x="69.85" y="26.67" smashed="yes" rot="R270">
 <attribute name="PROD_ID" value="TRANS-10060" x="69.85" y="26.67" size="1.778" layer="27" rot="R270" display="off"/>
 <attribute name="NAME" x="74.041" y="27.559" size="1.27" layer="25" font="vector" ratio="10"/>

Commit message: Added BOM. Minor changes to schematics and board.
Parts:
- C1, C2: value 47u -> 10u
Connections:
- net 5V: now also JP2.3
Routing:
- net 5V: track 115.5 -> 124.8 mm
Changed lines of the file:
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@@
 </autorouter>
 <elements>
-<element name="C1" library="SparkFun-Capacitors" package="CPOL-RADIAL-10UF-25V" value="47u" x="44.45" y="22.86" smashed="yes" rot="R90">
+<element name="C1" library="SparkFun-Capacitors" package="CPOL-RADIAL-10UF-25V" value="10u" x="44.45" y="22.86" smashed="yes" rot="R90">
 <attribute name="NAME" x="45.974" y="20.066" size="1.27" layer="25" font="vector" ratio="10" rot="R180"/>
 </element>
-<element name="C2" library="SparkFun-Capacitors" package="CPOL-RADIAL-10UF-25V" value="47u" x="44.45" y="29.21" smashed="yes">
+<element name="C2" library="SparkFun-Capacitors" package="CPOL-RADIAL-10UF-25V" value="10u" x="44.45" y="29.21" smashed="yes">
 <attribute name="NAME" x="43.561" y="25.654" size="1.27" layer="25" font="vector" ratio="10"/>
 </element>
@@
 <wire x1="23.495" y1="11.43" x2="39.37" y2="11.43" width="0.6096" layer="16"/>
 <wire x1="39.37" y1="11.43" x2="41.91" y2="13.97" width="0.6096" layer="16"/>
-<wire x1="41.91" y1="13.97" x2="41.91" y2="22.86" width="0.6096" layer="16"/>
+<wire x1="41.91" y1="13.97" x2="41.91" y2="20.32" width="0.6096" layer="16"/>
+<wire x1="41.91" y1="20.32" x2="41.91" y2="22.86" width="0.6096" layer="16"/>
 <wire x1="49.53" y1="21.59" x2="49.545" y2="17.78" width="0.6096" layer="1"/>
 <wire x1="49.545" y1="17.78" x2="59.69" y2="7.62" width="0.6096" layer="1"/>
@@
 <contactref element="C9" pad="1"/>
 <wire x1="16.51" y1="4.445" x2="16.51" y2="6.985" width="0.3048" layer="1"/>
+<contactref element="JP2" pad="3"/>
+<wire x1="34.29" y1="19.685" x2="34.29" y2="20.32" width="0.6096" layer="16"/>
+<wire x1="34.29" y1="20.32" x2="35.56" y2="21.59" width="0.6096" layer="16"/>
+<wire x1="35.56" y1="21.59" x2="40.64" y2="21.59" width="0.6096" layer="16"/>
+<wire x1="40.64" y1="21.59" x2="41.91" y2="20.32" width="0.6096" layer="16"/>
 </signal>
 <signal name="N$5">
